File: Emitter/Emitter.kicad_sch (KiCad schematic)
At the start: 2 parts, among them J1 Conn_01x02

Commit message: gnd fills
Connections:
- net GND: now reaches D1.1 (K), J1.1 (Pin_1)
Changed lines of the file:
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@@
 	(generator_version "8.0")
 	(paper "A4")
+	(junction
+		(at 49.53 55.88)
+		(diameter 0)
+		(color 0 0 0 0)
+	)
 	(wire
 		(pts
@@
 	(wire
 		(pts
-			(xy 54.61 55.88) (xy 46.99 55.88)
+			(xy 49.53 55.88) (xy 46.99 55.88)
 		)
 		(stroke
@@
 		)
 	)
+	(wire
+		(pts
+			(xy 54.61 55.88) (xy 49.53 55.88)
+		)
+		(stroke
+			(width 0)
+			(type default)
+		)
+	)
+	(symbol
+		(lib_id "power:GND")
+		(at 49.53 55.88 0)
+		(unit 1)
+		(exclude_from_sim no)
+		(in_bom yes)
+		(on_board yes)
+		(dnp no)
+		(fields_autoplaced yes)
+		(property "Reference" "#PWR01"
+			(at 49.53 62.23 0)
+			(effects
+				(font
+					(size 1.27 1.27)
+				)
+				(hide yes)
+			)
+		)
+		(property "Value" "GND"
+			(at 49.53 60.96 0)
+			(effects
+				(font
+					(size 1.27 1.27)
+				)
+			)
+		)
+		(property "Footprint" ""
+			(at 49.53 55.88 0)
+			(effects
+				(font
+					(size 1.27 1.27)
+				)
+				(hide yes)
+			)
+		)
+		(property "Datasheet" ""
+			(at 49.53 55.88 0)
+			(effects
+				(font
+					(size 1.27 1.27)
+				)
+				(hide yes)
+			)
+		)
+		(property "Description" "Power symbol creates a global label with name \"GND\" , ground"
+			(at 49.53 55.88 0)
+			(effects
+				(font
+					(size 1.27 1.27)
+				)
+				(hide yes)
+			)
+		)
+		(pin "1"
+		)
+		(instances
+			(project "Emitter"
+				(path "/14a34d3d-937f-4bd8-b41b-2dd62862cf47"
+					(reference "#PWR01")
+					(unit 1)
+				)
+			)
+		)
+	)
